File: MultiRJ45forRS485.kicad_sch (KiCad schematic)
At the start: 0 parts

Commit message: Create PCB
Parts:
- added H1, H2: MountingHole_Pad, MountingHole:MountingHole_4.3mm_M4_DIN965_Pad_TopOnly, symbol Mechanical:MountingHole_Pad
- added J1: Screw_Terminal_01x02, TerminalBlock:TerminalBlock_Altech_AK300-2_P5.00mm, symbol Connector:Screw_Terminal_01x02
- added U1: RJ45_56LED_2*2, PcbLib:RJ45_56LED_2*2, symbol SchLib:RJ45_56LED_2*2
Connections:
- new net: H1.1, H2.1, U1.0 (Shld)
- new net: J1.1 (Pin_1), U1.A1, U1.A3, U1.A5, U1.A7, U1.B1, U1.B3, U1.B5, U1.B7, U1.C1, U1.C3, U1.C5, U1.C7, U1.D1, U1.D3, U1.D5, U1.D7
- new net: J1.2 (Pin_2), U1.A2, U1.A4, U1.A6, U1.A8, U1.B2, U1.B4, U1.B6, U1.B8, U1.C2, U1.C4, U1.C6, U1.C8, U1.D2, U1.D4, U1.D6, U1.D8
- no-connect marks 0 -> 16
